File: V1/relay-24v-8ch-12a-v1.kicad_sch (KiCad schematic)
At the start: 44 parts, among them J1 DB141V-2.54-6P, J2 DB141V-2.54-6P, J3 DB142V-5.08-8P, J4 DB142V-5.08-8P, K1 G5PZ-1A, K2 G5PZ-1A, K3 G5PZ-1A, K4 G5PZ-1A, K5 G5PZ-1A, K6 G5PZ-1A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

Commit message: Updated connectors
Parts:
- removed J1, J2: DB141V-2.54-6P, Tales:TerminalBlock_Dibo_DB141V-2.54-6P_1x06_P2.54mm_Vertical, symbol Connector_Generic:Conn_01x06
- removed J3, J4: DB142V-5.08-8P, Tales:TerminalBlock_Dibo_DB142V-5.08-8P_1x08_P5.08mm_Vertical, symbol Connector_Generic:Conn_01x08
- added J1: DB141V-2.54-2P, Tales:TerminalBlock_Dibo_DB141V-2.54-2P_1x02_P2.54mm_Vertical, symbol Connector_Generic:Conn_01x02
- added J2, J3: DB141V-2.54-4P, Tales:TerminalBlock_Dibo_DB141V-2.54-4P_1x04_P2.54mm_Vertical, symbol Connector_Generic:Conn_01x04
- added J4, J5, J6, J7: DB142V-5.08-4P, Tales:TerminalBlock_Dibo_DB142V-5.08-4P_1x04_P5.08mm_Vertical, symbol Connector_Generic:Conn_01x04
- R1, R2, R3, R4, R5, R6, R7, R8: value 5k6/100mW -> 6k8/100mW; LCSC Part # C23189 -> C23212; Mfr PN 0603WAF5601T5E -> 0603WAF6801T5E; Vendor PN C23189 -> C23212
Connections:
- net +24V: now also J1.1 (Pin_1), J1.2 (Pin_2)
- net at D13.1 (K), D14.2 (A), K7.4: now also J3.2 (Pin_2)
- net at K5.2, RV5.1: now also J6.1 (Pin_1)
- net at K5.3, RV5.2: now also J6.2 (Pin_2)
- net at D7.1 (K), D8.2 (A), K4.4: now also J2.1 (Pin_1)
- net at K7.2, RV7.1: now also J7.1 (Pin_1)
- net at K7.3, RV7.2: now also J7.2 (Pin_2)
- net at K3.2, RV3.1: now also J5.1 (Pin_1)
- net at K3.3, RV3.2: now also J5.2 (Pin_2)
- net at D5.1 (K), D6.2 (A), K3.4: now also J2.2 (Pin_2)
- net at D1.1 (K), D2.2 (A), K1.4: now also J2.4 (Pin_4)
- net at D11.1 (K), D12.2 (A), K6.4: now also J3.3 (Pin_3)
- net at D10.2 (A), D9.1 (K), K5.4: now also J3.4 (Pin_4)
- net at K4.2, RV4.1: now also J5.3 (Pin_3)
- net at K4.3, RV4.2: now also J5.4 (Pin_4)
- net at D15.1 (K), D16.2 (A), K8.4: now also J3.1 (Pin_1)
- net at K6.2, RV6.1: now also J6.3 (Pin_3)
- net at K6.3, RV6.2: now also J6.4 (Pin_4)
- net at K8.2, RV8.1: now also J7.3 (Pin_3)
- net at K8.3, RV8.2: now also J7.4 (Pin_4)
- net at K1.2, RV1.1: now also J4.1 (Pin_1)
- net at K1.3, RV1.2: now also J4.2 (Pin_2)
- net at K2.2, RV2.1: now also J4.3 (Pin_3)
- net at K2.3, RV2.2: now also J4.4 (Pin_4)
- net at D3.1 (K), D4.2 (A), K2.4: now also J2.3 (Pin_3)
