File: V1/eumesmo-rl-8ch12a-v1.kicad_pcb (KiCad board)
At the start: 2 copper layers, 98 x 67.8 mm, 48 parts, among them J1 250-202, J2 250-204, J3 250-204, J4 DB142V-5.08-4P, J5 DB142V-5.08-4P, J6 DB142V-5.08-4P, J7 DB142V-5.08-4P, K1 G5PZ-1A, K2 G5PZ-1A, K3 G5PZ-1A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

Commit message: Release V1.2.0
Other:
- board text added: "V1.1 2026-06-17"
- board text removed: "V1.1 2026-06-12"
