File: V1/eumesmo-rl-8ch12a-v1.kicad_pcb (KiCad board)
At the start: 2 copper layers, 98 x 67.8 mm, 48 parts, among them J1 250-202, J2 250-204, J3 250-204, J4 DB142V-5.08-4P, J5 DB142V-5.08-4P, J6 DB142V-5.08-4P, J7 DB142V-5.08-4P, K1 G5PZ-1A, K2 G5PZ-1A, K3 G5PZ-1A, K4 G5PZ-1A, K5 G5PZ-1A, K6 G5PZ-1A, K7 G5PZ-1A, K8 G5PZ-1A

Commit message: Replaced 0603 size 10k resistor for 0805 size.
Parts:
- R1, R2, R3, R4, R5, R6, R7, R8: value 10k/100mW -> 10k/125mW; footprint Tales:R_0603_1608Metric -> Tales:R_0805_2012Metric
- moved R1 1.50 mm to (151.2, 67.0)
- moved R5 1.27 mm to (194.2, 64.8)
- moved R2 1.00 mm to (151.2, 69.0)
- moved R6 0.79 mm to (194.2, 66.8)
- moved R3 0.50 mm to (151.2, 71.0)
- moved R7 0.35 mm to (194.2, 68.8)
- moved R8 0.35 mm to (194.2, 70.8)
Routing:
- net +24V: track 231.2 -> 220.1 mm, vias 0 -> 2
- net /LED8: track 3.72 -> 2.79 mm
- net /LED1: track 21.3 -> 21.8 mm

Commit message: LEDs replaced for orange
Parts:
- D1, D11, D13, D15, D3, D5, D7, D9: value GREEN -> ORANGE/0603
Changed lines of the file:
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@@
 			)
 		)
-		(property "Value" "GREEN"
+		(property "Value" "ORANGE/0603"
 			(at 0 1.43 0)
 			(layer "F.Fab")
@@
 			)
 		)
-		(property "Mfr" "Everlight"
+		(property "Mfr" "Everlight Elec"
 			(at 0 0 0)
 			(unlocked yes)
@@
 			)
 		)
-		(property "Mfr PN" "19-217/GHC-YR1S2/3T"
+		(property "Mfr PN" "19-217/S2C-AL1M2VY/6T"
 			(at 0 0 0)
 			(unlocked yes)
@@
 			)
 		)
-		(property "Vendor PN" "C72043"
+		(property "Vendor PN" "C2987557"
 			(at 0 0 0)
 			(unlocked yes)
@@
 			)
 		)
-		(property "LCSC Part #" "C72043"
+		(property "LCSC Part #" "C2987557"
 			(at 0 0 0)
 			(unlocked yes)
@@
 			)
 		)
-		(property "Value" "GREEN"
+		(property "Value" "ORANGE/0603"
 			(at 0 1.43 0)
 			(layer "F.Fab")
@@
 			)
 		)
-		(property "LCSC Part #" "C72043"
+		(property "LCSC Part #" "C2987557"
 			(at 0 0 0)
 			(layer "F.Fab")
@@
 			)
 		)
-		(property "Mfr" "Everlight"
+		(property "Mfr" "Everlight Elec"
 			(at 0 0 0)
 			(layer "F.Fab")
@@
 			)
 		)
-		(property "Mfr PN" "19-217/GHC-YR1S2/3T"
+		(property "Mfr PN" "19-217/S2C-AL1M2VY/6T"
 			(at 0 0 0)
 			(layer "F.Fab")
@@
 			)
 		)
-		(property "Vendor PN" "C72043"
+		(property "Vendor PN" "C2987557"
 			(at 0 0 0)
 			(layer "F.Fab")
@@
 			)
 		)
-		(property "Value" "GREEN"
+		(property "Value" "ORANGE/0603"
 			(at 0 1.43 0)
 			(layer "F.Fab")
@@
 			)
 		)
-		(property "LCSC Part #" "C72043"
+		(property "LCSC Part #" "C2987557"
 			(at 0 0 0)
 			(layer "F.Fab")
@@
 			)
 		)
-		(property "Mfr" "Everlight"
+		(property "Mfr" "Everlight Elec"
 			(at 0 0 0)
 			(layer "F.Fab")
@@
 			)
 		)
-		(property "Mfr PN" "19-217/GHC-YR1S2/3T"
+		(property "Mfr PN" "19-217/S2C-AL1M2VY/6T"
 			(at 0 0 0)
 			(layer "F.Fab")
@@
 			)
 		)
-		(property "Vendor PN" "C72043"
+		(property "Vendor PN" "C2987557"
 			(at 0 0 0)
 			(layer "F.Fab")
@@
 			)
 		)
-		(property "Value" "GREEN"
+		(property "Value" "ORANGE/0603"
 			(at 0 1.43 0)
 			(layer "F.Fab")
@@
 			)
 		)
-		(property "Mfr" "Everlight"
+		(property "Mfr" "Everlight Elec"
 			(at 0 0 0)
 			(unlocked yes)
@@
 			)
 		)
-		(property "Mfr PN" "19-217/GHC-YR1S2/3T"
+		(property "Mfr PN" "19-217/S2C-AL1M2VY/6T"
 			(at 0 0 0)
 			(unlocked yes)
@@
 			)
 		)
-		(property "Vendor PN" "C72043"
+		(property "Vendor PN" "C2987557"
 			(at 0 0 0)
 			(unlocked yes)
@@
 			)
 		)
-		(property "LCSC Part #" "C72043"
+		(property "LCSC Part #" "C2987557"
 			(at 0 0 0)
 			(unlocked yes)
@@
 			)
 		)
-		(property "Value" "GREEN"
+		(property "Value" "ORANGE/0603"
 			(at 0 1.43 0)
 			(layer "F.Fab")
@@
 			)
 		)
-		(property "LCSC Part #" "C72043"
+		(property "LCSC Part #" "C2987557"
 			(at 0 0 0)
 			(layer "F.Fab")
@@
 			)
 		)
-		(property "Mfr" "Everlight"
+		(property "Mfr" "Everlight Elec"
 			(at 0 0 0)
 			(layer "F.Fab")
@@
 			)
 		)
-		(property "Mfr PN" "19-217/GHC-YR1S2/3T"
+		(property "Mfr PN" "19-217/S2C-AL1M2VY/6T"
 			(at 0 0 0)
 			(layer "F.Fab")
@@
 			)
 		)
-		(property "Vendor PN" "C72043"
+		(property "Vendor PN" "C2987557"
 			(at 0 0 0)
 			(layer "F.Fab")
@@
 			)
 		)
-		(property "Value" "GREEN"
+		(property "Value" "ORANGE/0603"
 			(at 0 1.43 0)
 			(layer "F.Fab")
@@
 			)
 		)
-		(property "Mfr" "Everlight"
+		(property "Mfr" "Everlight Elec"
 			(at 0 0 0)
 			(unlocked yes)
@@
 			)
 		)
-		(property "Mfr PN" "19-217/GHC-YR1S2/3T"
+		(property "Mfr PN" "19-217/S2C-AL1M2VY/6T"
 			(at 0 0 0)
 			(unlocked yes)
@@
 			)
 		)
-		(property "Vendor PN" "C72043"
+		(property "Vendor PN" "C2987557"
 			(at 0 0 0)
 			(unlocked yes)
@@
 			)
 		)
-		(property "LCSC Part #" "C72043"
+		(property "LCSC Part #" "C2987557"
 			(at 0 0 0)
 			(unlocked yes)
@@
 			)
 		)
-		(property "Value" "GREEN"
+		(property "Value" "ORANGE/0603"
 			(at 0 1.43 0)
 			(layer "F.Fab")
@@
 			)
 		)
-		(property "LCSC Part #" "C72043"
+		(property "LCSC Part #" "C2987557"
 			(at 0 0 0)
 			(layer "F.Fab")
@@
 			)
 		)
-		(property "Mfr" "Everlight"
+		(property "Mfr" "Everlight Elec"
 			(at 0 0 0)
 			(layer "F.Fab")
@@
 			)
 		)
-		(property "Mfr PN" "19-217/GHC-YR1S2/3T"
+		(property "Mfr PN" "19-217/S2C-AL1M2VY/6T"
 			(at 0 0 0)
 			(layer "F.Fab")
@@
 			)
 		)
-		(property "Vendor PN" "C72043"
+		(property "Vendor PN" "C2987557"
 			(at 0 0 0)
 			(layer "F.Fab")
@@
 			)
 		)
-		(property "Value" "GREEN"
+		(property "Value" "ORANGE/0603"
 			(at 0 1.43 0)
 			(layer "F.Fab")
@@
 			)
 		)
-		(property "Mfr" "Everlight"
+		(property "Mfr" "Everlight Elec"
 			(at 0 0 0)
 			(unlocked yes)
@@
 			)
 		)
-		(property "Mfr PN" "19-217/GHC-YR1S2/3T"
+		(property "Mfr PN" "19-217/S2C-AL1M2VY/6T"
 			(at 0 0 0)
 			(unlocked yes)
@@
 			)
 		)
-		(property "Vendor PN" "C72043"
+		(property "Vendor PN" "C2987557"
 			(at 0 0 0)
 			(unlocked yes)
@@
 			)
 		)
-		(property "LCSC Part #" "C72043"
+		(property "LCSC Part #" "C2987557"
 			(at 0 0 0)
 			(unlocked yes)
