File: V1/eumesmo-rl-8ch12a-v1.kicad_sch (KiCad schematic)
At the start: 47 parts, among them J1 250-202, J2 250-204, J3 250-204, J4 DB142V-5.08-4P, J5 DB142V-5.08-4P, J6 DB142V-5.08-4P, J7 DB142V-5.08-4P, K1 G5PZ-1A, K2 G5PZ-1A, K3 G5PZ-1A, K4 G5PZ-1A, K5 G5PZ-1A, K6 G5PZ-1A, K7 G5PZ-1A, K8 G5PZ-1A

Commit message: Replaced 0603 size 10k resistor for 0805 size.
Parts:
- R1, R2, R3, R4, R5, R6, R7, R8: value 10k/100mW -> 10k/125mW; footprint Tales:R_0603_1608Metric -> Tales:R_0805_2012Metric; LCSC Part # C25804 -> C17414; Mfr UNI-ROYAL(Uniroyal Elec) -> Uniroyal; Mfr PN 0603WAF1002T5E -> 0805W8F1002T5E; Package 0603/1608 -> 0805/2012; Vendor PN C25804 -> C17414
Changed lines of the file:
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@@
 			)
 		)
-		(property "Value" "10k/100mW"
+		(property "Value" "10k/125mW"
 			(at 171.45 110.49 0)
 			(show_name no)
@@
 			)
 		)
-		(property "Footprint" "Tales:R_0603_1608Metric"
+		(property "Footprint" "Tales:R_0805_2012Metric"
 			(at 175.006 110.744 90)
 			(hide yes)
@@
 			)
 		)
-		(property "Mfr" "UNI-ROYAL(Uniroyal Elec)"
+		(property "Mfr" "Uniroyal"
 			(at 173.99 110.49 0)
 			(hide yes)
@@
 			)
 		)
-		(property "Mfr PN" "0603WAF1002T5E"
+		(property "Mfr PN" "0805W8F1002T5E"
 			(at 173.99 110.49 0)
 			(hide yes)
@@
 			)
 		)
-		(property "Vendor PN" "C25804"
+		(property "Vendor PN" "C17414"
 			(at 173.99 110.49 0)
 			(hide yes)
@@
 			)
 		)
-		(property "LCSC Part #" "C25804"
+		(property "LCSC Part #" "C17414"
 			(at 171.45 113.03 0)
 			(show_name no)
@@
 			)
 		)
-		(property "Package" "0603/1608"
+		(property "Package" "0805/2012"
 			(at 173.99 110.49 0)
 			(hide yes)
@@
 			)
 		)
-		(property "Value" "10k/100mW"
+		(property "Value" "10k/125mW"
 			(at 171.45 148.59 0)
 			(show_name no)
@@
 			)
 		)
-		(property "Footprint" "Tales:R_0603_1608Metric"
+		(property "Footprint" "Tales:R_0805_2012Metric"
 			(at 175.006 148.844 90)
 			(hide yes)
@@
 			)
 		)
-		(property "Mfr" "UNI-ROYAL(Uniroyal Elec)"
+		(property "Mfr" "Uniroyal"
 			(at 173.99 148.59 0)
 			(hide yes)
@@
 			)
 		)
-		(property "Mfr PN" "0603WAF1002T5E"
+		(property "Mfr PN" "0805W8F1002T5E"
 			(at 173.99 148.59 0)
 			(hide yes)
@@
 			)
 		)
-		(property "Vendor PN" "C25804"
+		(property "Vendor PN" "C17414"
 			(at 173.99 148.59 0)
 			(hide yes)
@@
 			)
 		)
-		(property "LCSC Part #" "C25804"
+		(property "LCSC Part #" "C17414"
 			(at 171.45 151.13 0)
 			(show_name no)
@@
 			)
 		)
-		(property "Package" "0603/1608"
+		(property "Package" "0805/2012"
 			(at 173.99 148.59 0)
 			(hide yes)
@@
 			)
 		)
-		(property "Value" "10k/100mW"
+		(property "Value" "10k/125mW"
 			(at 73.66 31.75 0)
 			(show_name no)
@@
 			)
 		)
-		(property "Footprint" "Tales:R_0603_1608Metric"
+		(property "Footprint" "Tales:R_0805_2012Metric"
 			(at 77.216 32.004 90)
 			(hide yes)
@@
 			)
 		)
-		(property "Mfr" "UNI-ROYAL(Uniroyal Elec)"
+		(property "Mfr" "Uniroyal"
 			(at 76.2 31.75 0)
 			(hide yes)
@@
 			)
 		)
-		(property "Mfr PN" "0603WAF1002T5E"
+		(property "Mfr PN" "0805W8F1002T5E"
 			(at 76.2 31.75 0)
 			(hide yes)
@@
 			)
 		)
-		(property "Vendor PN" "C25804"
+		(property "Vendor PN" "C17414"
 			(at 76.2 31.75 0)
 			(hide yes)
@@
 			)
 		)
-		(property "LCSC Part #" "C25804"
+		(property "LCSC Part #" "C17414"
 			(at 73.66 34.29 0)
 			(show_name no)
@@
 			)
 		)
-		(property "Package" "0603/1608"
+		(property "Package" "0805/2012"
 			(at 76.2 31.75 0)
 			(hide yes)
@@
 			)
 		)
-		(property "Value" "10k/100mW"
+		(property "Value" "10k/125mW"
 			(at 73.66 107.95 0)
 			(show_name no)
@@
 			)
 		)
-		(property "Footprint" "Tales:R_0603_1608Metric"
+		(property "Footprint" "Tales:R_0805_2012Metric"
 			(at 77.216 108.204 90)
 			(hide yes)
@@
 			)
 		)
-		(property "Mfr" "UNI-ROYAL(Uniroyal Elec)"
+		(property "Mfr" "Uniroyal"
 			(at 76.2 107.95 0)
 			(hide yes)
@@
 			)
 		)
-		(property "Mfr PN" "0603WAF1002T5E"
+		(property "Mfr PN" "0805W8F1002T5E"
 			(at 76.2 107.95 0)
 			(hide yes)
@@
 			)
 		)
-		(property "Vendor PN" "C25804"
+		(property "Vendor PN" "C17414"
 			(at 76.2 107.95 0)
 			(hide yes)
@@
 			)
 		)
-		(property "LCSC Part #" "C25804"
+		(property "LCSC Part #" "C17414"
 			(at 73.66 110.49 0)
 			(show_name no)
@@
 			)
 		)
-		(property "Package" "0603/1608"
+		(property "Package" "0805/2012"
 			(at 76.2 107.95 0)
 			(hide yes)
@@
 			)
 		)
-		(property "Value" "10k/100mW"
+		(property "Value" "10k/125mW"
 			(at 73.66 69.85 0)
 			(show_name no)
@@
 			)
 		)
-		(property "Footprint" "Tales:R_0603_1608Metric"
+		(property "Footprint" "Tales:R_0805_2012Metric"
 			(at 77.216 70.104 90)
 			(hide yes)
@@
 			)
 		)
-		(property "Mfr" "UNI-ROYAL(Uniroyal Elec)"
+		(property "Mfr" "Uniroyal"
 			(at 76.2 69.85 0)
 			(hide yes)
@@
 			)
 		)
-		(property "Mfr PN" "0603WAF1002T5E"
+		(property "Mfr PN" "0805W8F1002T5E"
 			(at 76.2 69.85 0)
 			(hide yes)
@@
 			)
 		)
-		(property "Vendor PN" "C25804"
+		(property "Vendor PN" "C17414"
 			(at 76.2 69.85 0)
 			(hide yes)
@@
 			)
 		)
-		(property "LCSC Part #" "C25804"
+		(property "LCSC Part #" "C17414"
 			(at 73.66 72.39 0)
 			(show_name no)
@@
 			)
 		)
-		(property "Package" "0603/1608"
+		(property "Package" "0805/2012"
 			(at 76.2 69.85 0)
 			(hide yes)
@@
 			)
 		)
-		(property "Value" "10k/100mW"
+		(property "Value" "10k/125mW"
 			(at 171.45 72.39 0)
 			(show_name no)
@@
 			)
 		)
-		(property "Footprint" "Tales:R_0603_1608Metric"
+		(property "Footprint" "Tales:R_0805_2012Metric"
 			(at 175.006 72.644 90)
 			(hide yes)
@@
 			)
 		)
-		(property "Mfr" "UNI-ROYAL(Uniroyal Elec)"
+		(property "Mfr" "Uniroyal"
 			(at 173.99 72.39 0)
 			(hide yes)
@@
 			)
 		)
-		(property "Mfr PN" "0603WAF1002T5E"
+		(property "Mfr PN" "0805W8F1002T5E"
 			(at 173.99 72.39 0)
 			(hide yes)
@@
 			)
 		)
-		(property "Vendor PN" "C25804"
+		(property "Vendor PN" "C17414"
 			(at 173.99 72.39 0)
 			(hide yes)
@@
 			)
 		)
-		(property "LCSC Part #" "C25804"
+		(property "LCSC Part #" "C17414"
 			(at 171.45 74.93 0)
 			(show_name no)
@@
 			)
 		)
-		(property "Package" "0603/1608"
+		(property "Package" "0805/2012"
 			(at 173.99 72.39 0)
 			(hide yes)
@@
 			)
 		)
-		(property "Value" "10k/100mW"
+		(property "Value" "10k/125mW"
 			(at 73.66 146.05 0)
 			(show_name no)
@@
 			)
 		)
-		(property "Footprint" "Tales:R_0603_1608Metric"
+		(property "Footprint" "Tales:R_0805_2012Metric"
 			(at 77.216 146.304 90)
 			(hide yes)
@@
 			)
 		)
-		(property "Mfr" "UNI-ROYAL(Uniroyal Elec)"
+		(property "Mfr" "Uniroyal"
 			(at 76.2 146.05 0)
 			(hide yes)
@@
 			)
 		)
-		(property "Mfr PN" "0603WAF1002T5E"
+		(property "Mfr PN" "0805W8F1002T5E"
 			(at 76.2 146.05 0)
 			(hide yes)
@@
 			)
 		)
-		(property "Vendor PN" "C25804"
+		(property "Vendor PN" "C17414"
 			(at 76.2 146.05 0)
 			(hide yes)
@@
 			)
 		)
-		(property "LCSC Part #" "C25804"
+		(property "LCSC Part #" "C17414"
 			(at 73.66 148.59 0)
 			(show_name no)
@@
 			)
 		)
-		(property "Package" "0603/1608"
+		(property "Package" "0805/2012"
 			(at 76.2 146.05 0)
 			(hide yes)
@@
 			)
 		)
-		(property "Value" "10k/100mW"
+		(property "Value" "10k/125mW"
 			(at 171.45 34.29 0)
 			(show_name no)
@@
 			)
 		)
-		(property "Footprint" "Tales:R_0603_1608Metric"
+		(property "Footprint" "Tales:R_0805_2012Metric"
 			(at 175.006 34.544 90)
 			(hide yes)
@@
 			)
 		)
-		(property "Mfr" "UNI-ROYAL(Uniroyal Elec)"
+		(property "Mfr" "Uniroyal"
 			(at 173.99 34.29 0)
 			(hide yes)
@@
 			)
 		)
-		(property "Mfr PN" "0603WAF1002T5E"
+		(property "Mfr PN" "0805W8F1002T5E"
 			(at 173.99 34.29 0)
 			(hide yes)
@@
 			)
 		)
-		(property "Vendor PN" "C25804"
+		(property "Vendor PN" "C17414"
 			(at 173.99 34.29 0)
 			(hide yes)
@@
 			)
 		)
-		(property "LCSC Part #" "C25804"
+		(property "LCSC Part #" "C17414"
 			(at 171.45 36.83 0)
 			(show_name no)
@@
 			)
 		)
-		(property "Package" "0603/1608"
+		(property "Package" "0805/2012"
 			(at 173.99 34.29 0)
 			(hide yes)

Commit message: LEDs replaced for orange
Parts:
- D1, D11, D13, D15, D3, D5, D7, D9: value GREEN -> ORANGE/0603; LCSC Part # C72043 -> C2987557; Mfr Everlight -> Everlight Elec; Mfr PN 19-217/GHC-YR1S2/3T -> 19-217/S2C-AL1M2VY/6T; Vendor PN C72043 -> C2987557
Other:
- note added: "V_{F} = 1,8V @ 2,5mA I_{LED} = (24V - V_{F}) / R I_{LED} = (24V - 1.8V) / 10k I_{LED} = 2.22 mA"
Changed lines of the file:
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@@
 		(rev "V1.2")
 	)
+	(text "V_{F} = 1,8V @ 2,5mA\nI_{LED} = (24V - V_{F}) / R\nI_{LED} = (24V - 1.8V) / 10k\nI_{LED} = 2.22 mA"
+		(exclude_from_sim no)
+		(at 63.5 177.8 0)
+		(effects
+			(font
+				(size 1.5 1.5)
+			)
+			(justify left bottom)
+		)
+	)
 	(junction
 		(at 220.98 59.69)
@@
 			)
 		)
-		(property "Value" "GREEN"
+		(property "Value" "ORANGE/0603"
 			(at 73.66 156.21 90)
 			(show_name no)
@@
 			)
 		)
-		(property "Mfr" "Everlight"
+		(property "Mfr" "Everlight Elec"
 			(at 76.2 156.21 0)
 			(hide yes)
@@
 			)
 		)
-		(property "Mfr PN" "19-217/GHC-YR1S2/3T"
+		(property "Mfr PN" "19-217/S2C-AL1M2VY/6T"
 			(at 76.2 156.21 0)
 			(hide yes)
@@
 			)
 		)
-		(property "Vendor PN" "C72043"
+		(property "Vendor PN" "C2987557"
 			(at 76.2 156.21 0)
 			(hide yes)
@@
 			)
 		)
-		(property "LCSC Part #" "C72043"
+		(property "LCSC Part #" "C2987557"
 			(at 73.66 158.75 90)
 			(show_name no)
@@
 			)
 		)
-		(property "Value" "GREEN"
+		(property "Value" "ORANGE/0603"
 			(at 171.45 82.55 90)
 			(show_name no)
@@
 			)
 		)
-		(property "Mfr" "Everlight"
+		(property "Mfr" "Everlight Elec"
 			(at 173.99 82.55 0)
 			(hide yes)
@@
 			)
 		)
-		(property "Mfr PN" "19-217/GHC-YR1S2/3T"
+		(property "Mfr PN" "19-217/S2C-AL1M2VY/6T"
 			(at 173.99 82.55 0)
 			(hide yes)
@@
 			)
 		)
-		(property "Vendor PN" "C72043"
+		(property "Vendor PN" "C2987557"
 			(at 173.99 82.55 0)
 			(hide yes)
@@
 			)
 		)
-		(property "LCSC Part #" "C72043"
+		(property "LCSC Part #" "C2987557"
 			(at 171.45 85.09 90)
 			(show_name no)
@@
 			)
 		)
-		(property "Value" "GREEN"
+		(property "Value" "ORANGE/0603"
 			(at 73.66 118.11 90)
 			(show_name no)
@@
 			)
 		)
-		(property "Mfr" "Everlight"
+		(property "Mfr" "Everlight Elec"
 			(at 76.2 118.11 0)
 			(hide yes)
@@
 			)
 		)
-		(property "Mfr PN" "19-217/GHC-YR1S2/3T"
+		(property "Mfr PN" "19-217/S2C-AL1M2VY/6T"
 			(at 76.2 118.11 0)
 			(hide yes)
@@
 			)
 		)
-		(property "Vendor PN" "C72043"
+		(property "Vendor PN" "C2987557"
 			(at 76.2 118.11 0)
 			(hide yes)
@@
 			)
 		)
-		(property "LCSC Part #" "C72043"
+		(property "LCSC Part #" "C2987557"
 			(at 73.66 120.65 90)
 			(show_name no)
@@
 			)
 		)
-		(property "Value" "GREEN"
+		(property "Value" "ORANGE/0603"
 			(at 73.66 80.01 90)
 			(show_name no)
@@
 			)
 		)
-		(property "Mfr" "Everlight"
+		(property "Mfr" "Everlight Elec"
 			(at 76.2 80.01 0)
 			(hide yes)
@@
 			)
 		)
-		(property "Mfr PN" "19-217/GHC-YR1S2/3T"
+		(property "Mfr PN" "19-217/S2C-AL1M2VY/6T"
 			(at 76.2 80.01 0)
 			(hide yes)
@@
 			)
 		)
-		(property "Vendor PN" "C72043"
+		(property "Vendor PN" "C2987557"
 			(at 76.2 80.01 0)
 			(hide yes)
@@
 			)
 		)
-		(property "LCSC Part #" "C72043"
+		(property "LCSC Part #" "C2987557"
 			(at 73.66 82.55 90)
 			(show_name no)
@@
 			)
 		)
-		(property "Value" "GREEN"
+		(property "Value" "ORANGE/0603"
 			(at 171.45 158.75 90)
 			(show_name no)
@@
 			)
 		)
-		(property "Mfr" "Everlight"
+		(property "Mfr" "Everlight Elec"
 			(at 173.99 158.75 0)
 			(hide yes)
@@
 			)
 		)
-		(property "Mfr PN" "19-217/GHC-YR1S2/3T"
+		(property "Mfr PN" "19-217/S2C-AL1M2VY/6T"
 			(at 173.99 158.75 0)
 			(hide yes)
@@
 			)
 		)
-		(property "Vendor PN" "C72043"
+		(property "Vendor PN" "C2987557"
 			(at 173.99 158.75 0)
 			(hide yes)
@@
 			)
 		)
-		(property "LCSC Part #" "C72043"
+		(property "LCSC Part #" "C2987557"
 			(at 171.45 161.29 90)
 			(show_name no)
@@
 			)
 		)
-		(property "Value" "GREEN"
+		(property "Value" "ORANGE/0603"
 			(at 73.66 41.91 90)
 			(show_name no)
@@
 			)
 		)
-		(property "Mfr" "Everlight"
+		(property "Mfr" "Everlight Elec"
 			(at 76.2 41.91 0)
 			(hide yes)
@@
 			)
 		)
-		(property "Mfr PN" "19-217/GHC-YR1S2/3T"
+		(property "Mfr PN" "19-217/S2C-AL1M2VY/6T"
 			(at 76.2 41.91 0)
 			(hide yes)
@@
 			)
 		)
-		(property "Vendor PN" "C72043"
+		(property "Vendor PN" "C2987557"
 			(at 76.2 41.91 0)
 			(hide yes)
@@
 			)
 		)
-		(property "LCSC Part #" "C72043"
+		(property "LCSC Part #" "C2987557"
 			(at 73.66 44.45 90)
 			(show_name no)
@@
 			)
 		)
-		(property "Value" "GREEN"
+		(property "Value" "ORANGE/0603"
 			(at 171.45 120.65 90)
 			(show_name no)
@@
 			)
 		)
-		(property "Mfr" "Everlight"
+		(property "Mfr" "Everlight Elec"
 			(at 173.99 120.65 0)
 			(hide yes)
@@
 			)
 		)
-		(property "Mfr PN" "19-217/GHC-YR1S2/3T"
+		(property "Mfr PN" "19-217/S2C-AL1M2VY/6T"
 			(at 173.99 120.65 0)
 			(hide yes)
@@
 			)
 		)
-		(property "Vendor PN" "C72043"
+		(property "Vendor PN" "C2987557"
 			(at 173.99 120.65 0)
 			(hide yes)
@@
 			)
 		)
-		(property "LCSC Part #" "C72043"
+		(property "LCSC Part #" "C2987557"
 			(at 171.45 123.19 90)
 			(show_name no)
@@
 			)
 		)
-		(property "Value" "GREEN"
+		(property "Value" "ORANGE/0603"
 			(at 171.45 44.45 90)
 			(show_name no)
@@
 			)
 		)
-		(property "Mfr" "Everlight"
+		(property "Mfr" "Everlight Elec"
 			(at 173.99 44.45 0)
 			(hide yes)
@@
 			)
 		)
-		(property "Mfr PN" "19-217/GHC-YR1S2/3T"
+		(property "Mfr PN" "19-217/S2C-AL1M2VY/6T"
 			(at 173.99 44.45 0)
 			(hide yes)
@@
 			)
 		)
-		(property "Vendor PN" "C72043"
+		(property "Vendor PN" "C2987557"
 			(at 173.99 44.45 0)
 			(hide yes)
@@
 			)
 		)
-		(property "LCSC Part #" "C72043"
+		(property "LCSC Part #" "C2987557"
 			(at 171.45 46.99 90)
 			(show_name no)
